File: PCB-jig/epapertagjig-cam.brd (EAGLE design)
At the start: 98.5 x 79.9 mm, 53 parts, among them J1 CORTEX_JTAG_DEBUG_PTH, J10 CORTEX_JTAG_DEBUG_PTH, J21 CORTEX_JTAG_DEBUG_PTH, J4 CORTEX_JTAG_DEBUG_PTH, J6 JTAG, J7 CORTEX_JTAG_DEBUG_PTH, J9 ESP32-S3_DEVKITC-1, Q1 1.1A/60V/600mΩ, Q2 5.8A/30V/35mΩ, Q3 1.1A/60V/600mΩ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

Commit message: fixed mistake in PCB
Routing:
- net N$41: track 5.79 -> 70.4 mm, vias 0 -> 2
Changed lines of the file:
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@@
 <wire x1="56.261" y1="70.383" x2="56.261" y2="72.898" width="0.4064" layer="1"/>
 <wire x1="56.261" y1="72.898" x2="56.363" y2="72.898" width="0.4064" layer="1"/>
+<wire x1="53.086" y1="70.383" x2="53.086" y2="72.517" width="0.4064" layer="1"/>
+<via x="53.086" y="72.517" extent="1-16" drill="0.35"/>
+<wire x1="53.086" y1="72.517" x2="53.086" y2="68.707" width="0.4064" layer="16"/>
+<wire x1="53.086" y1="68.707" x2="53.848" y2="67.945" width="0.4064" layer="16"/>
+<wire x1="53.848" y1="67.945" x2="60.8838" y2="67.945" width="0.4064" layer="16"/>
+<wire x1="60.8838" y1="67.945" x2="63.5" y2="67.945" width="0.2032" layer="16"/>
+<wire x1="63.5" y1="67.945" x2="72.898" y2="67.945" width="0.4064" layer="16"/>
+<wire x1="72.898" y1="67.945" x2="73.66" y2="67.183" width="0.4064" layer="16"/>
+<wire x1="73.66" y1="67.183" x2="73.66" y2="47.498" width="0.4064" layer="16"/>
+<wire x1="73.66" y1="47.498" x2="82.55" y2="38.608" width="0.4064" layer="16"/>
+<via x="82.55" y="38.608" extent="1-16" drill="0.35"/>
+<wire x1="82.55" y1="38.608" x2="82.55" y2="38.735" width="0.4064" layer="1"/>
+<wire x1="82.55" y1="38.735" x2="87.63" y2="38.735" width="0.4064" layer="1"/>
 </signal>
 <signal name="N$42">
@@
 <mfgpreviewcolor name="substratecolor" color="0xFF786E46"/>
 </mfgpreviewcolors>
+<errors>
+</errors>
 </board>
 </drawing>
