File: PCB-jig/epapertagjig.sch (EAGLE design)
At the start: 48 parts, among them J1 CORTEX_JTAG_DEBUG_PTH, J10 CORTEX_JTAG_DEBUG_PTH, J4 CORTEX_JTAG_DEBUG_PTH, J6 JTAG, J7 CORTEX_JTAG_DEBUG_PTH, J9 ESP32-S3_DEVKITC-1, Q1 1.1A/60V/600mΩ, Q2 5.8A/30V/35mΩ, Q3 1.1A/60V/600mΩ, Q4 5.8A/30V/35mΩ

Commit message: fixed mistake in PCB
Connections:
- net N$41: now also J9.BOOT/0
Changed lines of the file:
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@@
 <wire x1="-10.16" y1="124.46" x2="-10.16" y2="144.78" width="0.1524" layer="91"/>
 <junction x="-10.16" y="144.78"/>
+<wire x1="-10.16" y1="124.46" x2="-10.16" y2="86.36" width="0.1524" layer="91"/>
+<wire x1="-10.16" y1="86.36" x2="132.08" y2="86.36" width="0.1524" layer="91"/>
+<junction x="-10.16" y="124.46"/>
+<pinref part="J9" gate="G$1" pin="BOOT/0"/>
+<wire x1="132.08" y1="86.36" x2="132.08" y2="53.34" width="0.1524" layer="91"/>
+<wire x1="132.08" y1="53.34" x2="124.46" y2="53.34" width="0.1524" layer="91"/>
 </segment>
 </net>
